File: status_beacon.kicad_sch (KiCad schematic)
At the start: 59 parts, among them J1 USB_C_16P, J2 SWD_TC2030, SW1 K2-1187SQ-A4SW-06, U1 PY32F003F18P6TU

Commit message: Close the release terminus: build, validate and commit fabrication outputs
Declare the artifact, archive, assembly, release-generation, reports and
release-profile blocks the build and release gates read, carry LCSC into the
schematic so the BOM the assembly house reads comes from the design authority,
and add the geometry tolerances the export-parity gates bound their comparisons
with. 18 gates pass, 15 report NOT_APPLICABLE with a reason.

Co-Authored-By: Claude Opus 5 <noreply@anthropic.com>
Parts:
- C1: LCSC (none) -> C1779
- C10, C11, C12, C13, C14, C15, C16, C2, C3, C4, C5, C6, C7, C8, C9: LCSC (none) -> C1525
- D1, D10, D11, D12, D2, D3, D4, D5, D6, D7, D8, D9: LCSC (none) -> C2761795
- D13, D14, D15, D16: LCSC (none) -> C48260
- J1: LCSC (none) -> C165948
- R1, R2: LCSC (none) -> C25905
- R3: LCSC (none) -> C17477
- R4: LCSC (none) -> C25105
- R5: LCSC (none) -> C11702
- R6: LCSC (none) -> C25744
- SW1: LCSC (none) -> C92584
- U1: LCSC (none) -> C5379864

Commit message: Series Schottky, and move off the discontinued LED
R3 (0R) becomes D17, a 1N5819WS Schottky in the VBUS to +5V path: a JLCPCB
basic part at $0.0116 with 1 A rating and Vf <= 0.60 V at 1 A. D1-D12 move
from WS2812B-B/T, which JLCPCB flags discontinued, to WS2812B-V5/W. The MCU
is unchanged: PY32F003F18P6TU is already the x6 variant, 1.7-5.5 V, so it
spans the whole post-diode rail with 2.65 V to spare below it.

The declared rails are now what the parts and the source actually permit.
VBUS is 4.75-5.5 V, which is vSafe5V rather than a narrower claim, so
usb_source_range_coverage passes on the truth instead of failing on a
declaration that did not cover the source. +5V runs from 4.15 V - the source
minimum less the diode's maximum forward voltage - up to 5.5 V, because no
diode datasheet guarantees a MINIMUM forward voltage and so nothing bounds
the rail from above.

That is the whole trade, and the claim model now states it exactly: the LED
absolute-maximum margins read -0.2 V as a LOWER bound, so their verdicts are
UNKNOWN rather than FAIL. The evidence cannot prove the rail exceeds 5.3 V
and cannot prove it does not. Rules go from 1 FAIL / 34 PASS / 11 UNKNOWN to
0 FAIL / 23 PASS / 23 UNKNOWN.

The V5 datasheet is better than the one it replaces and supersedes three
numbers. Working current is 12 mA per channel, so 36 mA per LED where 60 mA
had been assumed, taking the ring from 0.468 A to 0.281 A on direct evidence.
The shortest data high time is 220 ns, not 400 ns. VIH eases to 0.63xVDD
while VIL tightens to an absolute 0.7 V, and there is no characterised supply
range at all, only a 5 V test point - so the droop scenario now asserts
against the 3.7 V absolute minimum, driven at the source minimum less the
diode's maximum drop, which makes its 4.104 V result a lower bound.

Two rules were too narrow to survive the swap and are generalised rather than
patched: probe_access looked for an R-prefixed supply link when what it means
is exactly one two-terminal element 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
Parts:
- removed R3: 0R, Resistor_SMD:R_0805_2012Metric, symbol Device:R
- added D17: 1N5819WS, Diode_SMD:D_SOD-323, symbol Device:D_Schottky
- D1, D10, D11, D12, D2, D3, D4, D5, D6, D7, D8, D9: value WS2812B-B/T -> WS2812B-V5/W; LCSC C2761795 -> C2874885; MPN WS2812B-B/T -> WS2812B-V5/W
Connections:
- net +5V: now also D17.1 (K)
- net VBUS: now also D17.2 (A)
Other:
- moved on the sheet: J1, J2, R1, R2

Commit message: Regulate the rail: ME6211C50 LDO replaces the series Schottky
D17 and its 2 mV of margin are gone. U2 is an ME6211C50M5G-N in SOT-23-5,
with C17 as its input capacitor on VBUS; C1 stays on the output. The rail is
now the regulator's specified band rather than a source minus a drop nobody
guarantees: 4.05 to 5.05 V, against the WS2812B-V5's 3.70 to 5.30 V absolute
range. High margin +250 mV comes off the datasheet's +/-1% output tolerance;
low margin +350 mV from its dropout extrapolated to the declared port budget
and derated for temperature.

That is the whole point of the change. The twelve LED absolute-maximum checks
no longer report UNKNOWN because a lower bound could not decide them; they
PASS on a specified number. Board rules go from 0 FAIL / 23 PASS / 23 UNKNOWN
to 0 FAIL / 36 PASS / 11 UNKNOWN, and the eleven that remain are the
WS2812B's unspecified DOUT levels, which no part choice can settle.

Three things the regulator broke, each fixed by deriving from the topology
rather than restating it. The +5V power flag became a second power-output pin
once VOUT actually drove the net, so it is gone and VBUS and GND keep theirs.
The inrush rule summed capacitance across a hardcoded VBUS-plus-5V domain,
which was right when a link joined them and wrong once a regulator separated
them; it now walks the nets reachable through series passives, so only C17
counts. The supply-link rule required a two-terminal bridge; it now accepts
any single part touching both rails.

The SOT-23-5 needs more of the service arc than the 0805 link it replaced,
so that group is re-spaced from 11 to 9 degrees and shifted to clear the
courtyard overlap the first attempt hit.

23 gates pass, 62 tests pass, $1.7356 per board at qty 50.

Co-Authored-By: Claude Opus 5 <noreply@anthropic.com>
Parts:
- removed D17: 1N5819WS, Diode_SMD:D_SOD-323, symbol Device:D_Schottky
- added C17: 4.7uF, Capacitor_SMD:C_0805_2012Metric, symbol Device:C
- added U2: ME6211C50M5G-N, Package_TO_SOT_SMD:SOT-23-5, symbol StatusBeacon:ME6211C50
Connections:
- net +5V: now also U2.5 (VOUT)
- net GND: now also C17.2, U2.2 (VSS)
- net VBUS: now also C17.1, U2.1 (VIN), U2.3 (CE)
- no-connect marks 20 -> 21
Other:
- moved on the sheet: C1, C10, C11, C12, C13, C14, C15, C16, C2, C3, C4, C5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
